Commit message: Add files via upload

File: scholar_navigation/scholar_slam_description/urdf/top_plate.xacro (robot description, xacro)
@@ -50,7 +50,4 @@
     </collision>
   </link>
-  <!--link
-    name="front_laser_base_link">
-  </link-->
   <joint
     name="front_laser_base_joint"
@@ -66,7 +63,4 @@
       xyz="0 0 0" />
   </joint>
-  <!--link
-    name="rear_laser_base_link">
-  </link-->
   <joint
     name="rear_laser_base_joint"
@@ -89,5 +83,5 @@
     type="fixed">
     <origin
-      xyz="0.27747 0.00013521 0.097"
+      xyz="0.26146 -0.0016291 0.216"
       rpy="0 0 0" />
     <parent
@@ -96,5 +90,5 @@
       link="camera_base_link" />
     <axis
-      xyz="0 0 1" />
+      xyz="0 0 0" />
   </joint>
    <gazebo reference="camera_base_link">
